Commit message: Add z position of camera and laser

File: urdf/robot_tf.urdf (robot description, URDF)
Before this commit: robot mattbot, 4 links, 3 joints
Joints:
- joint camera_joint: origin xyz=0.127 0 0 rpy=0 0 0 -> xyz=0.127 0 0.190 rpy=0 0 0

File: urdf/robot_tf_car.urdf (robot description, URDF)
Before this commit: robot mattbot, 4 links, 3 joints
Joints:
- joint camera_joint: origin xyz=0.127 0 0 rpy=0 0 0 -> xyz=0.127 0 0.764 rpy=0 0 0
- joint laser_joint: origin xyz=0 0 0.1864 rpy=0 0 0 -> xyz=0 0 0.998 rpy=0 0 0

Commit message: Finalize the urdf configs

File: urdf/robot_tf.urdf (robot description, URDF)
Before this commit: robot mattbot, 4 links, 3 joints
Joints:
- joint camera_joint: origin xyz=0.127 0 0.190 rpy=0 0 0 -> xyz=0.127 0 0.764 rpy=0 0 0
- joint laser_joint: origin xyz=0 0 0.1864 rpy=0 0 0 -> xyz=0 0 0.998 rpy=0 0 0

File: urdf/robot_tf_short.urdf (robot description, URDF)
Before this commit: robot mattbot, 4 links, 3 joints
Joints:
- joint base_joint: origin xyz=0.1243076 0 0.0224 rpy=0 0 0 -> xyz=0 0 0.0224 rpy=0 0 0
- joint camera_joint: origin xyz=0.127 0 0.764 rpy=3.1416 0 0 -> xyz=0.127 0 0.190 rpy=0 0 0
- joint laser_joint: origin xyz=0 0 0.998 rpy=0 0 0 -> xyz=0 0 0.1864 rpy=0 0 0
